File: 8031.sch (KiCad schematic (older format))
At the start: 11 parts, among them J1 Conn_01x08_Male, J2 Conn_01x08_Male, U1 8031-cache_8031-cache_8031, U2 74LS373, U3 27128, Y1 12M

Commit message: 8031b
Parts:
- removed J2: Conn_01x08_Male, Connector_PinHeader_2.54mm:PinHeader_1x08_P2.54mm_Vertical, symbol Connector:Conn_01x08_Male
- added C5: 103, symbol Device:C_Small
- added C6: 104, symbol Device:C_Small
- added C7: 100U, symbol Device:CP_Small
- added J2: Conn_01x04_Male, symbol Connector:Conn_01x04_Male
- added LS1: Speaker, symbol Device:Speaker
- added R2, R3: R_Small, symbol Device:R_Small
- added U4: NE555, symbol Timer:NE555
Connections:
- net GND: now also C5.1, C5.2, C6.2, J2.4 (Pin_4), LS1.2, R3.2, U4.1 (GND), U4.2 (TR), U4.6 (THR)
- net VCC: now also U1.40 (VCC), J2.1 (Pin_1), R2.1, U4.8 (VCC)
- net at U1.10 (RXD\P3.0): now also J2.2 (Pin_2)
- net at U1.11 (TXD\P3.1): now also J2.3 (Pin_3)
- net P3.5: now reaches U1.15 (T1\P3.5)
- net P3.5: now also U4.4 (R)
- new net: C7.1, U4.3 (Q)
- new net: R2.2, R3.1, U4.7 (DIS)
- new net: C6.1, C7.2, LS1.1
- no-connect marks 4 -> 8
Other:
- moved on the sheet: C3, C4, J1, R1
